Commit message: Updated stuff

File: ROS/src/general/pegasus_description/urdf/pegasus.urdf (robot description, URDF)
Before this commit: robot pegasus, 12 links, 11 joints
Joints:
- joint axis0_joint: type fixed -> continuous
- joint axis1_joint: type fixed -> continuous

Commit message: bump2

File: ROS/src/general/pegasus_description/urdf/pegasus.urdf (robot description, URDF)
Before this commit: robot pegasus, 12 links, 11 joints
Links:
- added link /ugr/car_base_link/axis_steering
Joints:
- removed joint axis0_joint
- removed joint axis1_joint
- added joint axis0: type continuous, parent /ugr/car_base_link, child /ugr/car_base_link/axis0, origin xyz=-0.36 0.34 0 rpy=0 0 0
- added joint axis1: type continuous, parent /ugr/car_base_link, child /ugr/car_base_link/axis1, origin xyz=-0.36 -0.34 0 rpy=0 0 0
- added joint axis_steering: type continuous, parent /ugr/car_base_link, child /ugr/car_base_link/axis_steering, origin xyz=0.36 0.0 0 rpy=0 0 0

Commit message: Added joint limits

File: ROS/src/general/pegasus_description/urdf/pegasus.urdf (robot description, URDF)
Before this commit: robot pegasus, 13 links, 12 joints
Joints:
- joint axis0: limit (none) -> effort=100.0 velocity=10.0
- joint axis_steering: limit (none) -> lower=-1.0 upper=1.0 effort=100.0 velocity=10.0; type continuous -> revolute

Commit message: Fixed small issues

File: ROS/src/general/pegasus_description/urdf/pegasus.urdf (robot description, URDF)
Before this commit: robot pegasus, 13 links, 12 joints
Joints:
- joint axis0: limit effort=100.0 velocity=10.0 -> effort=100.0 velocity=100.0
- joint axis_steering: limit lower=-1.0 upper=1.0 effort=100.0 velocity=10.0 -> lower=-1.5 upper=1.5 effort=100.0 velocity=10.0

Commit message: Fixed steering

File: ROS/src/general/pegasus_description/urdf/pegasus.urdf (robot description, URDF)
Before this commit: robot pegasus, 13 links, 12 joints
Joints:
- joint axis_steering: limit lower=-1.5 upper=1.5 effort=100.0 velocity=10.0 -> lower=-3.14 upper=3.14 effort=100.0 velocity=10.0

Commit message: Moved car base link backwards

File: ROS/src/general/pegasus_description/urdf/pegasus.urdf (robot description, URDF)
Before this commit: robot pegasus, 13 links, 12 joints
Joints:
- joint axis0: origin xyz=-0.36 0.34 0 rpy=0 0 0 -> xyz=0.0 0.34 0 rpy=0 0 0
- joint axis1: origin xyz=-0.36 -0.34 0 rpy=0 0 0 -> xyz=0.0 -0.34 0 rpy=0 0 0
- joint axis_steering: origin xyz=0.36 0.0 0 rpy=0 0 0 -> xyz=0.72 0.0 0 rpy=0 0 0
- joint cam0_joint: origin xyz=0.06 0 0.74 rpy=0 0 -0.0218149 -> xyz=0.42 0 0.74 rpy=0 0 -0.0218149
- joint gps_ublox_left_joint: origin xyz=0.06 0.36 0.74 rpy=0 0 0 -> xyz=0.42 0.36 0.74 rpy=0 0 0
- joint gps_ublox_right_joint: origin xyz=0.06 -0.36 0.74 rpy=0 0 0 -> xyz=0.42 -0.36 0.74 rpy=0 0 0
- joint imu0_joint: origin xyz=-0.26 0 0.35 rpy=0 0 0 -> xyz=0.10 0 0.35 rpy=0 0 0
- joint imu1_joint: origin xyz=-0.26 0 0.37 rpy=3.1415 0 0 -> xyz=0.10 0 0.37 rpy=3.1415 0 0
- joint lidar0_joint: origin xyz=0.0 0 0.37 rpy=0 0 0 -> xyz=0.36 0 0.37 rpy=0 0 0

Commit message: bump

File: ROS/src/general/pegasus_description/urdf/pegasus.urdf (robot description, URDF)
Before this commit: robot pegasus, 13 links, 12 joints
Links:
- removed link /ugr/car_base_link
- removed link /ugr/car_base_link/axis0
- removed link /ugr/car_base_link/axis1
- removed link /ugr/car_base_link/axis_steering
- removed link /ugr/car_base_link/cam0
- removed link /ugr/car_base_link/gps0
- removed link /ugr/car_base_link/gps1
- removed link /ugr/car_base_link/imu0
- removed link /ugr/car_base_link/imu1
- removed link /ugr/car_base_link/lidar0
- removed link /ugr/car_base_link/os_imu
- removed link /ugr/car_base_link/os_lidar
- removed link /ugr/car_base_link/os_sensor
- added link ugr/car_base_link
- added link ugr/car_base_link/axis0
- added link ugr/car_base_link/axis1
- added link ugr/car_base_link/axis_steering
- added link ugr/car_base_link/cam0
- added link ugr/car_base_link/gps0
- added link ugr/car_base_link/gps1
- added link ugr/car_base_link/imu0
- added link ugr/car_base_link/imu1
- added link ugr/car_base_link/lidar0
- added link ugr/car_base_link/os_imu
- added link ugr/car_base_link/os_lidar
- added link ugr/car_base_link/os_sensor
Joints:
- joint axis0: child /ugr/car_base_link/axis0 -> ugr/car_base_link/axis0; parent /ugr/car_base_link -> ugr/car_base_link
- joint axis1: child /ugr/car_base_link/axis1 -> ugr/car_base_link/axis1; parent /ugr/car_base_link -> ugr/car_base_link
- joint axis_steering: child /ugr/car_base_link/axis_steering -> ugr/car_base_link/axis_steering; parent /ugr/car_base_link -> ugr/car_base_link
- joint cam0_joint: child /ugr/car_base_link/cam0 -> ugr/car_base_link/cam0; parent /ugr/car_base_link -> ugr/car_base_link
- joint gps_ublox_left_joint: child /ugr/car_base_link/gps1 -> ugr/car_base_link/gps1; parent /ugr/car_base_link -> ugr/car_base_link
- joint gps_ublox_right_joint: child /ugr/car_base_link/gps0 -> ugr/car_base_link/gps0; parent /ugr/car_base_link -> ugr/car_base_link
- joint imu0_joint: child /ugr/car_base_link/imu0 -> ugr/car_base_link/imu0; parent /ugr/car_base_link -> ugr/car_base_link
- joint imu1_joint: child /ugr/car_base_link/imu1 -> ugr/car_base_link/imu1; parent /ugr/car_base_link -> ugr/car_base_link
- joint lidar0_joint: child /ugr/car_base_link/lidar0 -> ugr/car_base_link/lidar0; parent /ugr/car_base_link -> ugr/car_base_link
- joint os_imu_joint: child /ugr/car_base_link/os_imu -> ugr/car_base_link/os_imu; parent /ugr/car_base_link/os_sensor -> ugr/car_base_link/os_sensor
- joint os_lidar_joint: child /ugr/car_base_link/os_lidar -> ugr/car_base_link/os_lidar; parent /ugr/car_base_link/os_sensor -> ugr/car_base_link/os_sensor
- joint os_sensor_joint: child /ugr/car_base_link/os_sensor -> ugr/car_base_link/os_sensor; parent /ugr/car_base_link/lidar0 -> ugr/car_base_link/lidar0

Commit message: Made improveemnts to Pegasus model

File: ROS/src/general/pegasus_description/urdf/pegasus.urdf (robot description, URDF)
Before this commit: robot pegasus, 13 links, 12 joints
Joints:
- joint axis0: limit effort=100.0 velocity=100.0 -> effort=30.0 velocity=100.0
