Commit message: changes

File: ROS/src/orion_description/urdf/orion.urdf (robot description, URDF)
Before this commit: robot orion, 12 links, 11 joints
Joints:
- joint axis_rear: limit effort=30.0 velocity=100.0 -> effort=120.0 velocity=100.0

Commit message: lidar works, added frame for vizualisation

File: ROS/src/orion_description/urdf/orion.urdf (robot description, URDF)
Before this commit: robot orion, 12 links, 11 joints
Links:
- added link ugr/car_base_link/os_sensor_normal
Joints:
- added joint os_sensor_turn: type fixed, parent ugr/car_base_link/os_sensor, child ugr/car_base_link/os_sensor_normal, origin xyz=0 0 0 rpy=3.1415 0 0
- joint cam0_joint: origin xyz=0.6814 -0.0824 0.8230 rpy=0 0 3.1415 -> xyz=0.6814 -0.0824 0.8230 rpy=3.1415 0 0
- joint lidar0_joint: origin xyz=0.6765 -0.0022 0.7870 rpy=3.1415 0 0 -> xyz=0.6765 -0.0022 1.6450 rpy=3.1415 0 0

Commit message: can test

File: ROS/src/orion_description/urdf/orion.urdf (robot description, URDF)
Before this commit: robot orion, 12 links, 11 joints
Joints:
- joint cam0_joint: origin xyz=0.6814 -0.0824 0.8230 rpy=0 0 3.1415 -> xyz=0.6814 -0.0824 0.8230 rpy=0 0 0

Commit message: Fixed ros control (almost)

File: ROS/src/orion_description/urdf/orion.urdf (robot description, URDF)
Before this commit: robot orion, 12 links, 11 joints
Joints:
- joint axis_rear: limit effort=120.0 velocity=100.0 -> effort=60.0 velocity=100.0

Commit message: Added 2 frames

File: ROS/src/orion_description/urdf/orion.urdf (robot description, URDF)
Before this commit: robot orion, 12 links, 11 joints
Links:
- removed link ugr/car_base_link/axis_rear
- added link ugr/car_base_link/axis0
- added link ugr/car_base_link/axis1
Joints:
- removed joint axis_rear
- added joint axis0: type continuous, parent ugr/car_base_link, child ugr/car_base_link/axis0, origin xyz=0.0 -0.64 0.0 rpy=0 0 0, limit effort=60.0 velocity=100.0
- added joint axis1: type continuous, parent ugr/car_base_link, child ugr/car_base_link/axis1, origin xyz=0.0 0.64 0.0 rpy=0 0 0, limit effort=60.0 velocity=100.0

Commit message: remeasured

File: ROS/src/orion_description/urdf/orion.urdf (robot description, URDF)
Before this commit: robot orion, 13 links, 12 joints
Joints:
- joint lidar0_joint: origin xyz=0.6765 -0.0022 1.6450 rpy=3.1415 0 0 -> xyz=0.6765 -0.0022 0.78 rpy=3.1415 0 0

Commit message: comp fixes

File: ROS/src/orion_description/urdf/orion.urdf (robot description, URDF)
Before this commit: robot orion, 14 links, 13 joints
Joints:
- joint axis0: limit effort=60.0 velocity=100.0 -> effort=240.0 velocity=100.0
- joint axis1: limit effort=60.0 velocity=100.0 -> effort=240.0 velocity=100.0
