Commit message: change pegasus limits [VERIFY LATER]

File: ROS/src/pegasus_description/urdf/pegasus.urdf (robot description, URDF)
Before this commit: robot pegasus, 14 links, 13 joints
Joints:
- joint axis0: limit effort=30.0 velocity=100.0 -> effort=3000.0 velocity=10000.0

Commit message: working

File: ROS/src/pegasus_description/urdf/pegasus.urdf (robot description, URDF)
Before this commit: robot pegasus, 14 links, 13 joints
Joints:
- joint axis0: limit effort=3000.0 velocity=10000.0 -> effort=30.0 velocity=100.0

Commit message: massive dump of MPC code

File: ROS/src/pegasus_description/urdf/pegasus.urdf (robot description, URDF)
Before this commit: robot pegasus, 14 links, 13 joints
Joints:
- joint axis0: limit effort=30.0 velocity=100.0 -> effort=30.0 velocity=200.0

Commit message: forgot dvsv en increased pegasus limit

File: ROS/src/pegasus_description/urdf/pegasus.urdf (robot description, URDF)
Before this commit: robot pegasus, 14 links, 13 joints
Joints:
- joint axis0: limit effort=30.0 velocity=100.0 -> effort=30.0 velocity=1000.0

Commit message: revert urdf change bcs actually not save at all irl

File: ROS/src/pegasus_description/urdf/pegasus.urdf (robot description, URDF)
Before this commit: robot pegasus, 14 links, 13 joints
Joints:
- joint axis0: limit effort=30.0 velocity=1000.0 -> effort=30.0 velocity=100.0

Commit message: removed non mpc changes

File: ROS/src/pegasus_description/urdf/pegasus.urdf (robot description, URDF)
Before this commit: robot pegasus, 14 links, 13 joints
Joints:
- joint axis0: limit effort=30.0 velocity=200.0 -> effort=30.0 velocity=100.0
